Commit message: updates

File: urdf/gp7.urdf (robot description, URDF)
Before this commit: robot yaskawa_gp7, 10 links, 9 joints
Links:
- added link world
Joints:
- added joint world_fixed: type fixed, parent world, child base_link, origin xyz=0 0 0 rpy=0 0 0
- joint joint_b: axis 0 -1 0 -> 0 1 0; limit lower=-2.356 upper=2.356 effort=1 velocity=9.59 -> lower=-2.356 upper=2.356 effort=1000 velocity=9.59
- joint joint_l: limit lower=-1.134 upper=2.530 effort=1 velocity=5.49 -> lower=-1.134 upper=2.530 effort=1000 velocity=5.49
- joint joint_r: axis -1 0 0 -> 1 0 0; limit lower=-3.316 upper=3.316 effort=1 velocity=9.59 -> lower=-3.316 upper=3.316 effort=1000 velocity=9.59
- joint joint_s: limit lower=-2.967 upper=2.967 effort=1 velocity=6.54 -> lower=-2.967 upper=2.967 effort=1000 velocity=6.54
- joint joint_t: axis -1 0 0 -> 1 0 0; limit lower=-6.283 upper=6.283 effort=1 velocity=17.45 -> lower=-6.283 upper=6.283 effort=1000 velocity=17.45
- joint joint_u: axis 0 -1 0 -> 0 1 0; limit lower=-2.024 upper=4.450 effort=1 velocity=7.15 -> lower=-2.024 upper=4.450 effort=1000 velocity=7.15

Commit message: adding griper

File: urdf/gp7.urdf (robot description, URDF)
Before this commit: robot yaskawa_gp7, 11 links, 10 joints
Links:
- removed link gripper_link
- added link left_inner_knuckle, mass 0.01; visual mesh filename=package://gp7_sim/meshes/robotiq/visual/inner_knuckle_fine.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
- added link left_outer_finger, mass 0.02; collision mesh filename=package://gp7_sim/meshes/robotiq/collision/outer_finger_coa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; visual mesh filename=package://gp7_sim/meshes/robotiq/visual/outer_finger_fine.S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
- added link left_outer_knuckle, mass 0.01; collision mesh filename=package://gp7_sim/meshes/robotiq/collision/outer_knuckle_co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; visual mesh filename=package://gp7_sim/meshes/robotiq/visual/outer_knuckle_fine.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
- added link right_inner_knuckle, mass 0.01; visual mesh filename=package://gp7_sim/meshes/robotiq/visual/inner_knuckle_fine.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
- added link right_outer_finger, mass 0.02; collision mesh filename=package://gp7_sim/meshes/robotiq/collision/outer_finger_coa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; visual mesh filename=package://gp7_sim/meshes/robotiq/visual/outer_finger_fine.S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
- added link right_outer_knuckle, mass 0.01; collision mesh filename=package://gp7_sim/meshes/robotiq/collision/outer_knuckle_co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; visual mesh filename=package://gp7_sim/meshes/robotiq/visual/outer_knuckle_fine.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
- added link robotiq_85_base_link, mass 0.3; collision mesh filename=package://gp7_sim/meshes/robotiq/collision/robotiq_85_base_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; visual mesh filename=package://gp7_sim/meshes/robotiq/visual/robotiq_85_base_lin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
Joints:
- removed joint tool0_to_gripper
- added joint finger_joint: type fixed, parent robotiq_85_base_link, child left_outer_knuckle, origin xyz=0.0306 0 0.0627 rpy=0 0 0
- added joint flange_to_robotiq: type fixed, parent flange, child robotiq_85_base_link, origin xyz=0 0 0 rpy=0 0 0
- added joint left_inner_knuckle_joint: type fixed, parent robotiq_85_base_link, child left_inner_knuckle, origin xyz=0.0127 0 0.0693
- added joint left_outer_finger_joint: type fixed, parent left_outer_knuckle, child left_outer_finger, origin xyz=0.0316 0 -0.0019 rpy=0 0 0
- added joint right_inner_knuckle_joint: type fixed, parent robotiq_85_base_link, child right_inner_knuckle, origin xyz=-0.0127 0 0.0693 rpy=0 0 3.14159
- added joint right_outer_finger_joint: type fixed, parent right_outer_knuckle, child right_outer_finger, origin xyz=0.0316 0 -0.0016 rpy=0 0 0
- added joint right_outer_knuckle_joint: type fixed, parent robotiq_85_base_link, child right_outer_knuckle, origin xyz=-0.0306 0 0.0627 rpy=0 0 3.14159

Commit message: update arm

File: urdf/gp7.urdf (robot description, URDF)
Before this commit: robot yaskawa_gp7, 17 links, 16 joints
Links:
- removed link left_inner_knuckle
- removed link right_inner_knuckle
Joints:
- removed joint left_inner_knuckle_joint
- removed joint right_inner_knuckle_joint
- joint finger_joint: axis (none) -> 0 -1 0; limit (none) -> lower=0 upper=0.8 effort=1000 velocity=0.5; type fixed -> revolute
- joint right_outer_knuckle_joint: axis (none) -> 0 -1 0; limit (none) -> lower=0 upper=0.8 effort=1000 velocity=0.5; type fixed -> revolute

Commit message: finetuning grab mechanism

File: urdf/gp7.urdf (robot description, URDF)
Before this commit: robot yaskawa_gp7, 15 links, 14 joints
Joints:
- joint finger_joint: limit lower=0 upper=0.8 effort=1000 velocity=0.5 -> lower=0 upper=0.8 effort=100000 velocity=0.5
- joint right_outer_knuckle_joint: limit lower=0 upper=0.8 effort=1000 velocity=0.5 -> lower=0 upper=0.8 effort=100000 velocity=0.5
